Commit message: fixed an error

File: urdf/LSC16.urdf.xacro (robot description, xacro)
@@ -1,5 +1,5 @@
 <?xml version="1.0"?>
 <robot xmlns:xacro="http://www.ros.org/wiki/xacro" name="LSC16">
-  <xacro:macro name="LSC16" params="*origin parent:=base_link name:=velodyne">
+  <xacro:macro name="LSC16" params="*origin parent:=base_link name:=lslidar">
     <joint name="${name}_base_mount_joint" type="fixed">
       <xacro:insert_block name="origin" />

Commit message: removed inertial block

File: urdf/LSC16.urdf.xacro (robot description, xacro)
@@ -8,11 +8,4 @@
     </joint>
     <link name="${name}_base_link">
-      <inertial>
-        <mass value="0.83"/>
-        <origin xyz="0 0 0"/>
-        <inertia ixx="${(0.83 * (3.0*0.0516*0.0516 + 0.0717*0.0717)) / 12.0}" ixy="0" ixz="0"
-          iyy="${(0.83 * (3.0*0.0516*0.0516 + 0.0717*0.0717)) / 12.0}" iyz="0"
-          izz="${0.5 * 0.83 * (0.0516*0.0516)}"/>
-      </inertial>
       <visual>
         <geometry>
@@ -38,9 +31,4 @@
     </joint>
     <link name="${name}">
-      <inertial>
-        <mass value="0.01"/>
-        <origin xyz="0 0 0"/>
-        <inertia ixx="1e-7" ixy="0" ixz="0" iyy="1e-7" iyz="0" izz="1e-7"/>
-      </inertial>
       <visual>
         <origin xyz="0 0 0" />
